Commit message: Improved Navigation, goal recognition and marker visualization implemented

File: Software/jetson_racer/urdf/jetracer.xacro (robot description, xacro)
@@ -20,10 +20,10 @@
   <xacro:property name="deg_to_rad" value="0.01745329251994329577"/>
   <!-- Robot base dimensions -->
-  <xacro:property name="base_length" value="0.5" />
-  <xacro:property name="base_width" value="0.3" />
+  <xacro:property name="base_length" value="0.3" />
+  <xacro:property name="base_width" value="0.15" />
   <xacro:property name="base_height" value="0.1" />
   <xacro:property name="base_mass" value="5" />
   <!-- Wheel link dimensions -->
-  <xacro:property name="wheel_radius" value="0.1" />
+  <xacro:property name="wheel_radius" value="0.05" />
   <xacro:property name="wheel_thickness" value="0.08" />
   <xacro:property name="wheel_mass" value="1" />
